File: hardware/interfaces.kicad_sch (KiCad schematic)
At the start: 8 parts, among them J105 USB_C_Receptacle_USB2.0_14P, J106 CAN, U102 TJA1051T-3

Commit message: Layout work
Parts:
- J106: footprint Connector_JST:JST_GH_SM04B-GHS-TB_1x04-1MP_P1.25mm_Horizontal -> Connector_JST:JST_PH_B4B-PH-SM4-TB_1x04-1MP_P2.00mm_Vertical
Connections:
- net +5V: now also J106.4 (Pin_4); no longer J106.1 (Pin_1)
- net CAN_N: now also J106.2 (Pin_2); no longer J106.3 (Pin_3)
- net CAN_P: now also J106.3 (Pin_3); no longer J106.2 (Pin_2)
- net GND: now also J106.1 (Pin_1); no longer J106.4 (Pin_4)
Other:
- moved on the sheet: J106
Changed lines of the file:
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@@
+	)
+	(junction
+		(at 91.44 62.23)
+		(diameter 0)
+		(color 0 0 0 0)
 	)
 	(junction
@@
 	(wire
 		(pts
+			(xy 96.52 49.53) (xy 99.06 49.53)
+		)
+		(stroke
+			(width 0)
+			(type default)
+		)
+	)
+	(wire
+		(pts
 			(xy 49.53 63.5) (xy 49.53 68.58)
 		)
@@
 	(wire
 		(pts
+			(xy 93.98 62.23) (xy 93.98 64.77)
+		)
+		(stroke
+			(width 0)
+			(type default)
+		)
+	)
+	(wire
+		(pts
+			(xy 99.06 64.77) (xy 99.06 49.53)
+		)
+		(stroke
+			(width 0)
+			(type default)
+		)
+	)
+	(wire
+		(pts
 			(xy 139.7 63.5) (xy 139.7 66.04)
 		)
@@
 	(wire
 		(pts
+			(xy 93.98 64.77) (xy 99.06 64.77)
+		)
+		(stroke
+			(width 0)
+			(type default)
+		)
+	)
+	(wire
+		(pts
 			(xy 87.63 60.96) (xy 91.44 60.96)
 		)
@@
 		(pts
 			(xy 74.93 60.96) (xy 77.47 60.96)
+		)
+		(stroke
+			(width 0)
+			(type default)
+		)
+	)
+	(wire
+		(pts
+			(xy 91.44 62.23) (xy 93.98 62.23)
 		)
 		(stroke
@@
 	(symbol
 		(lib_id "power:GND")
-		(at 96.52 67.31 0)
-		(unit 1)
-		(exclude_from_sim no)
-		(in_bom yes)
-		(on_board yes)
-		(dnp no)
-		(fields_autoplaced yes)
-		(property "Reference" "#PWR0135"
-			(at 96.52 73.66 0)
-			(effects
-				(font
-					(size 1.27 1.27)
-				)
-				(hide yes)
-			)
-		)
-		(property "Value" "GND"
-			(at 96.52 72.39 0)
-			(effects
-				(font
-					(size 1.27 1.27)
-				)
-			)
-		)
-		(property "Footprint" ""
-			(at 96.52 67.31 0)
-			(effects
-				(font
-					(size 1.27 1.27)
-				)
-				(hide yes)
-			)
-		)
-		(property "Datasheet" ""
-			(at 96.52 67.31 0)
-			(effects
-				(font
-					(size 1.27 1.27)
-				)
-				(hide yes)
-			)
-		)
-		(property "Description" "Power symbol creates a global label with name \"GND\" , ground"
-			(at 96.52 67.31 0)
-			(effects
-				(font
-					(size 1.27 1.27)
-				)
-				(hide yes)
-			)
-		)
-		(pin "1"
-		)
-		(instances
-			(project "greenmobi-drive"
-				(path "/a12b77e7-bd0f-4a70-9ba2-19a87ce48819/9fd9bfb7-5a26-4f3a-8811-151b2a5ffd2d"
-					(reference "#PWR0135")
-					(unit 1)
-				)
-			)
-		)
-	)
-	(symbol
-		(lib_id "power:GND")
 		(at 50.8 40.64 0)
 		(unit 1)
@@
 	(symbol
 		(lib_id "Connector_Generic_MountingPin:Conn_01x04_MountingPin")
-		(at 96.52 57.15 0)
-		(unit 1)
-		(exclude_from_sim no)
-		(in_bom yes)
-		(on_board yes)
-		(dnp no)
-		(fields_autoplaced yes)
+		(at 96.52 59.69 0)
+		(mirror x)
+		(unit 1)
+		(exclude_from_sim no)
+		(in_bom yes)
+		(on_board yes)
+		(dnp no)
 		(property "Reference" "J106"
-			(at 99.06 57.5055 0)
+			(at 99.06 59.3345 0)
 			(effects
 				(font
@@
 		)
 		(property "Value" "CAN"
-			(at 99.06 60.0455 0)
+			(at 99.06 56.7945 0)
 			(effects
 				(font
@@
 			)
 		)
-		(property "Footprint" "Connector_JST:JST_GH_SM04B-GHS-TB_1x04-1MP_P1.25mm_Horizontal"
-			(at 96.52 57.15 0)
+		(property "Footprint" "Connector_JST:JST_PH_B4B-PH-SM4-TB_1x04-1MP_P2.00mm_Vertical"
+			(at 96.52 59.69 0)
 			(effects
 				(font
@@
 		)
 		(property "Datasheet" "~"
-			(at 96.52 57.15 0)
+			(at 96.52 59.69 0)
 			(effects
 				(font
@@
 		)
 		(property "Description" "Generic connectable mounting pin connector, single row, 01x04, script generated (kicad-library-utils/schlib/autogen/connector/)"
-			(at 96.52 57.15 0)
+			(at 96.52 59.69 0)
 			(effects
 				(font
@@
 		)
 		(property "LCSC" "C17700382"
-			(at 96.52 57.15 0)
-			(effects
-				(font
+			(at 96.52 59.69 0)
+			(effects
+				(font
